Commit message: feat(sim): add stack launcher and tune simulation performance
Add a host launcher and generated world with 14 dynamic obstacles. Support headless Gazebo, reduce the AGV footprint and sensor rates, and throttle odometry and TF with non-finite velocity guards.

Co-Authored-By: Claude Code <noreply@anthropic.com>

File: urdf/agv/agv.urdf.xacro (robot description, xacro)
@@ -6,11 +6,13 @@
     without touching anything else in this package.
   -->
-  <xacro:property name="base_length" value="0.60"/>
-  <xacro:property name="base_width"  value="0.50"/>
+  <!-- Body shrunk to 40 x 30 cm (from 60 x 50). Height and wheel radius stay
+       so the spawn height / wheel-ground contact geometry does not change. -->
+  <xacro:property name="base_length" value="0.40"/>
+  <xacro:property name="base_width"  value="0.30"/>
   <xacro:property name="base_height" value="0.25"/>
   <xacro:property name="wheel_radius" value="0.10"/>
   <xacro:property name="wheel_width"  value="0.04"/>
-  <xacro:property name="wheelbase" value="0.50"/>
-  <xacro:property name="track_width" value="0.42"/>
+  <xacro:property name="wheelbase" value="0.32"/>
+  <xacro:property name="track_width" value="0.26"/>
   <!-- base_footprint: standard Nav2 footprint frame (odom -> base_footprint -> base_link) -->
   <link name="base_footprint"/>
@@ -130,4 +132,6 @@
       <odom_frame>odom</odom_frame>
       <robot_base_frame>base_footprint</robot_base_frame>
+      <!-- OnUpdate runs at 1 kHz; publish odom/TF at a sane ROS rate. -->
+      <publish_rate>50.0</publish_rate>
     </plugin>
   </gazebo>
@@ -136,5 +140,5 @@
       <pose>0 0 0 0 0 0</pose>
       <visualize>true</visualize>
-      <update_rate>20.0</update_rate>
+      <update_rate>10.0</update_rate>
       <ray>
         <scan>
@@ -163,5 +167,5 @@
   <gazebo reference="camera_link">
     <sensor type="depth" name="camera_depth">
-      <update_rate>15.0</update_rate>
+      <update_rate>5.0</update_rate>
       <camera>
         <horizontal_fov>1.3962634</horizontal_fov>
@@ -180,5 +184,5 @@
   <gazebo reference="camera_link">
     <sensor type="camera" name="camera_color">
-      <update_rate>15.0</update_rate>
+      <update_rate>5.0</update_rate>
       <camera>
         <horizontal_fov>1.3962634</horizontal_fov>
@@ -195,22 +199,7 @@
     </sensor>
   </gazebo>
-  <!-- Aligned depth camera: same pose/intrinsics as color, publishes depth
-       registered to the color frame (required by hanmole dynamicDetector). -->
-  <gazebo reference="camera_link">
-    <sensor type="depth" name="camera_aligned_depth">
-      <update_rate>15.0</update_rate>
-      <camera>
-        <horizontal_fov>1.3962634</horizontal_fov>
-        <image><width>640</width><height>480</height></image>
-        <clip><near>0.1</near><far>20.0</far></clip>
-      </camera>
-      <plugin name="camera_aligned_depth_plugin" filename="libgazebo_ros_camera.so">
-        <ros>
-          <remapping>image_raw:=/camera/aligned_depth_to_color/image_raw</remapping>
-          <remapping>camera_info:=/camera/aligned_depth_to_color/camera_info</remapping>
-        </ros>
-        <frame_name>camera_link</frame_name>
-      </plugin>
-    </sensor>
-  </gazebo>
+  <!-- Aligned depth camera removed: the detector reads /camera_depth/depth/image_raw
+       directly (aligned_depth_image_topic points at the depth image), so this third
+       camera only doubled the software-rendering cost. Restore if a color-aligned
+       depth stream is ever needed. -->
 </robot>
