Commit message: feat(sim): mecanum AGV, /scan lidar, dynamic worlds and RViz config
- add mecanum drive plugin: cmd_vel -> four wheel speeds, odom and TF
- publish 2D lidar as /scan; add spawn_x/spawn_y args and stable spawn height
- port Intent-MPC generated_env worlds (static + dense dynamic obstacles)
- extend dynamic scenes with person/box models; add RViz and ground-truth updates
- drive wheels with velocity + fmax torque limit (no self-driving without cmd_vel)
- publish real odometry twist (body frame) instead of the commanded value

File: urdf/agv/agv.urdf.xacro (robot description, xacro)
@@ -2,5 +2,5 @@
 <robot xmlns:xacro="http://www.ros.org/wiki/xacro" name="agv">
   <!--
-    Minimal differential-drive AGV for nav_sim.
+    Minimal mecanum-wheel AGV for nav_sim.
     Stack-agnostic: publishes /scan, /odom, TF. Swap in your own URDF here
     without touching anything else in this package.
@@ -11,4 +11,13 @@
   <xacro:property name="wheel_radius" value="0.10"/>
   <xacro:property name="wheel_width"  value="0.04"/>
+  <xacro:property name="wheelbase" value="0.50"/>
+  <xacro:property name="track_width" value="0.42"/>
+  <!-- base_footprint: standard Nav2 footprint frame (odom -> base_footprint -> base_link) -->
+  <link name="base_footprint"/>
+  <joint name="base_footprint_joint" type="fixed">
+    <parent link="base_footprint"/>
+    <child link="base_link"/>
+    <origin xyz="0 0 0.05" rpy="0 0 0"/>
+  </joint>
   <!-- base_link -->
   <link name="base_link">
@@ -28,6 +37,6 @@
     </collision>
   </link>
-  <!-- chassis wheels (left/right), driven by diff drive plugin -->
-  <xacro:macro name="wheel" params="prefix side">
+  <!-- chassis wheels (4x mecanum), driven by mecanum_drive_plugin -->
+  <xacro:macro name="mecanum_wheel" params="prefix x y">
     <link name="${prefix}_wheel">
       <inertial>
@@ -49,10 +58,12 @@
       <parent link="base_link"/>
       <child link="${prefix}_wheel"/>
-      <origin xyz="${side * base_width/2} 0 -${wheel_radius}" rpy="0 0 0"/>
+      <origin xyz="${x} ${y} -${wheel_radius}" rpy="0 0 0"/>
       <axis xyz="0 1 0"/>
     </joint>
   </xacro:macro>
-  <xacro:wheel prefix="left" side="1.0"/>
-  <xacro:wheel prefix="right" side="-1.0"/>
+  <xacro:mecanum_wheel prefix="front_left"  x="${ wheelbase/2}" y="${ track_width/2}"/>
+  <xacro:mecanum_wheel prefix="front_right" x="${ wheelbase/2}" y="${-track_width/2}"/>
+  <xacro:mecanum_wheel prefix="rear_left"   x="${-wheelbase/2}" y="${ track_width/2}"/>
+  <xacro:mecanum_wheel prefix="rear_right"  x="${-wheelbase/2}" y="${-track_width/2}"/>
   <!-- caster (passive ball) -->
   <link name="caster_link">
@@ -104,19 +115,19 @@
   </gazebo>
   <gazebo>
-    <plugin name="diff_drive" filename="libgazebo_ros_diff_drive.so">
+    <plugin name="mecanum_drive" filename="libmecanum_drive_plugin.so">
       <ros>
         <remapping>cmd_vel:=/cmd_vel</remapping>
         <remapping>odom:=/odom</remapping>
       </ros>
-      <left_joint>left_wheel_joint</left_joint>
-      <right_joint>right_wheel_joint</right_joint>
-      <wheel_separation>${base_width}</wheel_separation>
-      <wheel_diameter>${2*wheel_radius}</wheel_diameter>
+      <front_left_joint>front_left_wheel_joint</front_left_joint>
+      <front_right_joint>front_right_wheel_joint</front_right_joint>
+      <rear_left_joint>rear_left_wheel_joint</rear_left_joint>
+      <rear_right_joint>rear_right_wheel_joint</rear_right_joint>
+      <wheel_radius>${wheel_radius}</wheel_radius>
+      <wheelbase>${wheelbase}</wheelbase>
+      <track_width>${track_width}</track_width>
       <max_wheel_torque>20.0</max_wheel_torque>
-      <max_wheel_acceleration>1.0</max_wheel_acceleration>
-      <publish_odom>true</publish_odom>
-      <publish_odom_tf>true</publish_odom_tf>
       <odom_frame>odom</odom_frame>
-      <robot_base_frame>base_link</robot_base_frame>
+      <robot_base_frame>base_footprint</robot_base_frame>
     </plugin>
   </gazebo>
@@ -143,5 +154,5 @@
       <plugin name="lidar_2d_plugin" filename="libgazebo_ros_ray_sensor.so">
         <ros>
-          <remapping>out:=/scan</remapping>
+          <remapping>/lidar_2d_plugin/out:=/scan</remapping>
         </ros>
         <output_type>sensor_msgs/LaserScan</output_type>
@@ -184,3 +195,22 @@
     </sensor>
   </gazebo>
+  <!-- Aligned depth camera: same pose/intrinsics as color, publishes depth
+       registered to the color frame (required by hanmole dynamicDetector). -->
+  <gazebo reference="camera_link">
+    <sensor type="depth" name="camera_aligned_depth">
+      <update_rate>15.0</update_rate>
+      <camera>
+        <horizontal_fov>1.3962634</horizontal_fov>
+        <image><width>640</width><height>480</height></image>
+        <clip><near>0.1</near><far>20.0</far></clip>
+      </camera>
+      <plugin name="camera_aligned_depth_plugin" filename="libgazebo_ros_camera.so">
+        <ros>
+          <remapping>image_raw:=/camera/aligned_depth_to_color/image_raw</remapping>
+          <remapping>camera_info:=/camera/aligned_depth_to_color/camera_info</remapping>
+        </ros>
+        <frame_name>camera_link</frame_name>
+      </plugin>
+    </sensor>
+  </gazebo>
 </robot>

Commit message: fix: fix sim config

File: urdf/agv/agv.urdf.xacro (robot description, xacro)
@@ -2,5 +2,5 @@
 <robot xmlns:xacro="http://www.ros.org/wiki/xacro" name="agv">
   <!--
-    Minimal mecanum-wheel AGV for nav_sim.
+    Planar omnidirectional navigation AGV for nav_sim.
     Stack-agnostic: publishes /scan, /odom, TF. Swap in your own URDF here
     without touching anything else in this package.
@@ -39,5 +39,5 @@
     </collision>
   </link>
-  <!-- chassis wheels (4x mecanum), driven by mecanum_drive_plugin -->
+  <!-- Fixed wheel geometry: planar_drive_plugin controls the rigid chassis. -->
   <xacro:macro name="mecanum_wheel" params="prefix x y">
     <link name="${prefix}_wheel">
@@ -57,10 +57,13 @@
       </collision>
     </link>
-    <joint name="${prefix}_wheel_joint" type="continuous">
+    <joint name="${prefix}_wheel_joint" type="fixed">
       <parent link="base_link"/>
       <child link="${prefix}_wheel"/>
       <origin xyz="${x} ${y} -${wheel_radius}" rpy="0 0 0"/>
-      <axis xyz="0 1 0"/>
     </joint>
+    <gazebo reference="${prefix}_wheel">
+      <mu1>0.01</mu1>
+      <mu2>0.01</mu2>
+    </gazebo>
   </xacro:macro>
   <xacro:mecanum_wheel prefix="front_left"  x="${ wheelbase/2}" y="${ track_width/2}"/>
@@ -111,26 +114,22 @@
     <origin xyz="${base_length/2 - 0.02} 0 ${base_height}" rpy="0 0 0"/>
   </joint>
-  <!-- Gazebo plugins: diff drive, lidar, camera -->
+  <!-- Gazebo plugins: planar drive, lidar, camera -->
   <gazebo reference="base_link">
     <material>Gazebo/Grey</material>
     <gravity>true</gravity>
   </gazebo>
+  <gazebo reference="caster_link">
+    <mu1>0.01</mu1>
+    <mu2>0.01</mu2>
+  </gazebo>
   <gazebo>
-    <plugin name="mecanum_drive" filename="libmecanum_drive_plugin.so">
+    <plugin name="planar_drive" filename="libplanar_drive_plugin.so">
       <ros>
         <remapping>cmd_vel:=/cmd_vel</remapping>
         <remapping>odom:=/odom</remapping>
       </ros>
-      <front_left_joint>front_left_wheel_joint</front_left_joint>
-      <front_right_joint>front_right_wheel_joint</front_right_joint>
-      <rear_left_joint>rear_left_wheel_joint</rear_left_joint>
-      <rear_right_joint>rear_right_wheel_joint</rear_right_joint>
-      <wheel_radius>${wheel_radius}</wheel_radius>
-      <wheelbase>${wheelbase}</wheelbase>
-      <track_width>${track_width}</track_width>
-      <max_wheel_torque>20.0</max_wheel_torque>
       <odom_frame>odom</odom_frame>
       <robot_base_frame>base_footprint</robot_base_frame>
-      <!-- OnUpdate runs at 1 kHz; publish odom/TF at a sane ROS rate. -->
+      <cmd_vel_timeout>0.5</cmd_vel_timeout>
       <publish_rate>50.0</publish_rate>
     </plugin>
